Commit message: ur support addition initiated + tests on coupled mobility

File: shadow_hand/robots/shadow_hand.srdf.xacro (robot description, xacro)
@@ -18,29 +18,3 @@
 		</xacro:if>
 	</xacro:macro>
-	<!-- <group_state group="right_hand" name="pack2">
-			<joint name="rh_THJ1" value="0.52" />
-			<joint name="rh_THJ2" value="0.61" />
-			<joint name="rh_THJ3" value="0.00" />
-			<joint name="rh_THJ4" value="1.20" />
-			<joint name="rh_THJ5" value="0.17" />
-			<joint name="rh_FFJ1" value="1.5707" />
-			<joint name="rh_FFJ2" value="1.5707" />
-			<joint name="rh_FFJ3" value="1.5707" />
-			<joint name="rh_FFJ4" value="0" />
-			<joint name="rh_MFJ1" value="1.5707" />
-			<joint name="rh_MFJ2" value="1.5707" />
-			<joint name="rh_MFJ3" value="1.5707" />
-			<joint name="rh_MFJ4" value="0" />
-			<joint name="rh_RFJ1" value="1.5707" />
-			<joint name="rh_RFJ2" value="1.5707" />
-			<joint name="rh_RFJ3" value="1.5707" />
-			<joint name="rh_RFJ4" value="0" />
-			<joint name="rh_LFJ1" value="1.5707" />
-			<joint name="rh_LFJ2" value="1.5707" />
-			<joint name="rh_LFJ3" value="1.5707" />
-			<joint name="rh_LFJ4" value="0" />
-			<joint name="rh_LFJ5" value="0" />
-			<joint name="rh_WRJ1" value="0" />
-			<joint name="rh_WRJ2" value="0" />
-	</group_state> -->
 </robot>

File: shadow_hand/robots/shadow_hand.urdf.xacro (robot description, xacro)
@@ -46,46 +46,11 @@
 		</plugin>
 	</gazebo> -->
-	<!-- ... new group state which uses shadow_finger xacros ......................................................... -->
-	<!-- <xacro:arg name="robot_name" default="shadowhand_motor" />
-	<xacro:arg name="hand_name" default="right_hand" />
-	<xacro:arg name="prefix" default="rh_" />
-	<xacro:arg name="ff" default="1" />
-	<xacro:arg name="mf" default="1" />
-	<xacro:arg name="rf" default="1" />
-	<xacro:arg name="lf" default="1" />
-	<xacro:arg name="th" default="1" />
-	<xacro:arg name="is_lite" default="0" />
-	<xacro:arg name="is_biotac" default="0" />
-	<group_state name="pack2" group="$(arg hand_name)">
-		<xacro:if value="$(arg th)">
-			<xacro:thumb_curl prefix="$(arg prefix)" is_biotac="$(arg is_biotac)" />
-		</xacro:if>
-		<xacro:if value="$(arg ff)">
-			<xacro:finger_curl prefix="$(arg prefix)" joint_prefix="FF" lf="0"
-				is_biotac="$(arg is_biotac)" />
-		</xacro:if>
-		<xacro:if value="$(arg mf)">
-			<xacro:finger_curl prefix="$(arg prefix)" joint_prefix="MF" lf="0"
-				is_biotac="$(arg is_biotac)" />
-		</xacro:if>
-		<xacro:if value="$(arg rf)">
-			<xacro:finger_curl prefix="$(arg prefix)" joint_prefix="RF" lf="0"
-				is_biotac="$(arg is_biotac)" />
-		</xacro:if>
-		<xacro:unless value="$(arg is_lite)">
-			<xacro:if value="$(arg lf)">
-				<xacro:finger_curl prefix="$(arg prefix)" joint_prefix="LF" lf="1"
-					is_biotac="$(arg is_biotac)" />
-			</xacro:if>
-			<joint name="$(arg prefix)WRJ1" value="0" />
-			<joint name="$(arg prefix)WRJ2" value="0" />
-		</xacro:unless>
-	</group_state> -->
-	<gazebo>
-		<plugin filename="libsim_biotac.so" name="sim_biotac">
+	<!-- <gazebo>
+		<plugin filename="libbiotac_sim_lib.so" name="biotac_sim">
 			<alwaysOn>true</alwaysOn>
 			<updateRate>100.0</updateRate>
-			<!-- <updateRate>100.0</updateRate> -->
 		</plugin>
-	</gazebo>
+	</gazebo> -->
 </robot>
+<!-- [Err] [Plugin.hh:212] Failed to load plugin libsim_biotac.so: libsim_biotac.so: cannot open shared object file: No such file or directory -->
+<!-- libbiotac_sim_lib.so -->
