Commit message: run robot and hand with different init poses

File: shadow_hand/robots/sr_hand.urdf.xacro (robot description, xacro)
@@ -31,4 +31,6 @@
   <xacro:include filename="$(find sr_description)/hand/xacro/hand.urdf.xacro"/>
   <xacro:include filename="$(find sr_description)/other/xacro/gazebo.urdf.xacro"/>
+  <xacro:arg name="initial_hand_position" default="0.0 0.0 1.0"/>
+  <xacro:arg name="initial_hand_orientation" default="1.57 -1.57 0.0"/>
   <xacro:arg name="hand_type" default="hand_e"/>
   <xacro:arg name="hand_version" default="E3M5"/>
@@ -45,5 +47,6 @@
       <parent link="world" />
       <child link="rh_forearm" />
-      <origin xyz="0.0 0.0 0.0" rpy="0.0 0.0 0.0" />
+      <origin xyz="$(arg initial_hand_position)" rpy="$(arg initial_hand_orientation)" />
+      <!-- <origin xyz="0.0 0.0 1.0" rpy="0.0 0.0 0.0" /> -->
     </joint>
   </xacro:if>
@@ -52,5 +55,6 @@
       <parent link="world" />
       <child link="lh_forearm" />
-      <origin xyz="0.0 0.0 0.0" rpy="0.0 0.0 0.0" />
+      <origin xyz="$(arg initial_hand_position)" rpy="$(arg initial_hand_orientation)" />
+      <!-- <origin xyz="0.0 0.0 0.0" rpy="0.0 0.0 0.0" /> -->
     </joint>
   </xacro:if>

File: shadow_hand/robots/srhand_ur.urdf.xacro (robot description, xacro)
@@ -28,10 +28,5 @@
        xmlns:interface="http://playerstage.sourceforge.net/gazebo/xmlschema/#interface" name="ursrh">
     <link name="world"/>
-    <xacro:arg name="initial_x" default="0.0"/>
-    <xacro:arg name="initial_y" default="0.0"/>
-    <xacro:arg name="initial_z" default="0.0"/>
-    <xacro:arg name="initial_R" default="0.0"/>
-    <xacro:arg name="initial_P" default="0.0"/>
-    <xacro:arg name="initial_Y" default="0.0"/>
+    <!-- -x 0.0 -y 0.0 -z 0.1 -R 0.0 -P 0.0 -Y 0.0 -->
     <xacro:arg name="transmission_hw_interface" default="hardware_interface/PositionJointInterface"/>
     <xacro:arg name="robot_model" default="ur10e"/>
@@ -46,4 +41,6 @@
     <xacro:arg name="prox_sensors" default="none"/>
     <xacro:arg name="palm_sensor" default="none"/>
+    <xacro:arg name="initial_robot_position" default="0.0 0.0 0.1"/>
+    <xacro:arg name="initial_robot_orientation" default="0.0 0.0 0.0"/>
     <xacro:if value="${'$(arg side)' == 'right'}">
         <xacro:arg name="arm_prefix" default="ra" />
@@ -75,5 +72,6 @@
         <parent link="world"/>
         <child link="$(arg arm_prefix)_base_link"/>
-        <origin xyz="$(arg initial_x) $(arg initial_y) $(arg initial_z)" rpy="$(arg initial_R) $(arg initial_P) $(arg initial_Y)"/>
+        <origin xyz="$(arg initial_robot_position)" rpy="$(arg initial_robot_orientation)"/>
+        <!-- <origin xyz="$(arg initial_x) $(arg initial_y) $(arg initial_z)" rpy="$(arg initial_R) $(arg initial_P) $(arg initial_Y)"/> -->
     </joint>
     <joint name="$(arg arm_prefix)_arm_to_hand" type="fixed">
