Commit message: launch file complete refactorisation

File: shadow_hand/robots/shadow_hand.urdf.xacro (robot description, xacro)
@@ -36,14 +36,8 @@
 		prox_sensors="$(arg prox_sensors)" palm_sensor="$(arg palm_sensor)"
 		mounting_plate="$(arg mounting_plate)" />
-	<!-- <link name="world" /> -->
-	<!-- <joint name="rh_world_joint" type="fixed">
-		<parent link="world" />
-		<child link="rh_forearm" />
-		<origin xyz="0.0 0.0 0.0" rpy="0.0 0.0 0.0" />
-	</joint> -->
 	<gazebo>
-		<plugin filename="libsim_biotac.so" name="sim_biotac">
-			<alwaysOn>
-				true</alwaysOn>
+		<!-- <plugin filename="libbiotac_sim_lib.so" name="biotac_sim_lib"> This works for some reason?! -->
+			<plugin filename="libsim_biotac.so" name="sim_biotac">
+			<alwaysOn>true</alwaysOn>
 			<updateRate>100.0</updateRate>
 		</plugin>

Commit message: improved real time joint control in ShadowHnad

File: shadow_hand/robots/shadow_hand.urdf.xacro (robot description, xacro)
@@ -4,4 +4,7 @@
 	xmlns:interface="http://playerstage.sourceforge.net/gazebo/xmlschema/#interface"
 	name="shadowhand_motor">
+	<!-- include local xacro file -->
+	<!-- <xacro:include filename="$(find shadow_hand)/robots/shadow_finger.srdf.xacro" /> -->
+	<!-- <xacro:include filename="$(find shadow_hand)/robots/shadowhand.srdf.xacro" /> -->
 	<xacro:include filename="$(find sr_description)/other/xacro/materials.urdf.xacro" />
 	<xacro:include filename="$(find sr_description)/hand/xacro/hand.urdf.xacro" />
@@ -36,5 +39,5 @@
 		prox_sensors="$(arg prox_sensors)" palm_sensor="$(arg palm_sensor)"
 		mounting_plate="$(arg mounting_plate)" />
-		<!-- <plugin filename="libbiotac_sim_lib.so" name="biotac_sim_lib"> This works for some reason?! -->
+	<!-- <plugin filename="libbiotac_sim_lib.so" name="biotac_sim_lib"> This works for some reason?! -->
 	<!-- <gazebo>
 		<plugin filename="libbiotac_sim_lib.so" name="biotac_sim_lib">
@@ -43,6 +46,42 @@
 		</plugin>
 	</gazebo> -->
+	<!-- ... new group state which uses shadow_finger xacros ......................................................... -->
+	<!-- <xacro:arg name="robot_name" default="shadowhand_motor" />
+	<xacro:arg name="hand_name" default="right_hand" />
+	<xacro:arg name="prefix" default="rh_" />
+	<xacro:arg name="ff" default="1" />
+	<xacro:arg name="mf" default="1" />
+	<xacro:arg name="rf" default="1" />
+	<xacro:arg name="lf" default="1" />
+	<xacro:arg name="th" default="1" />
+	<xacro:arg name="is_lite" default="0" />
+	<xacro:arg name="is_biotac" default="0" />
+	<group_state name="pack2" group="$(arg hand_name)">
+		<xacro:if value="$(arg th)">
+			<xacro:thumb_curl prefix="$(arg prefix)" is_biotac="$(arg is_biotac)" />
+		</xacro:if>
+		<xacro:if value="$(arg ff)">
+			<xacro:finger_curl prefix="$(arg prefix)" joint_prefix="FF" lf="0"
+				is_biotac="$(arg is_biotac)" />
+		</xacro:if>
+		<xacro:if value="$(arg mf)">
+			<xacro:finger_curl prefix="$(arg prefix)" joint_prefix="MF" lf="0"
+				is_biotac="$(arg is_biotac)" />
+		</xacro:if>
+		<xacro:if value="$(arg rf)">
+			<xacro:finger_curl prefix="$(arg prefix)" joint_prefix="RF" lf="0"
+				is_biotac="$(arg is_biotac)" />
+		</xacro:if>
+		<xacro:unless value="$(arg is_lite)">
+			<xacro:if value="$(arg lf)">
+				<xacro:finger_curl prefix="$(arg prefix)" joint_prefix="LF" lf="1"
+					is_biotac="$(arg is_biotac)" />
+			</xacro:if>
+			<joint name="$(arg prefix)WRJ1" value="0" />
+			<joint name="$(arg prefix)WRJ2" value="0" />
+		</xacro:unless>
+	</group_state> -->
 	<gazebo>
-			<plugin filename="libsim_biotac.so" name="sim_biotac">
+		<plugin filename="libsim_biotac.so" name="sim_biotac">
 			<alwaysOn>true</alwaysOn>
 			<updateRate>100.0</updateRate>

Commit message: go to mujoco v2.0

File: shadow_hand/robots/shadow_hand.urdf.xacro (robot description, xacro)
@@ -21,4 +21,5 @@
 	<link name="world" />
 	<xacro:if value="${'$(arg side)' == 'right'}">
+		<!-- <joint name="rh_world_joint" type="floating"> -->
 		<joint name="rh_world_joint" type="fixed">
 			<parent link="world" />

File: shadow_hand/robots/sr_hand.urdf.xacro (robot description, xacro)
@@ -31,5 +31,6 @@
   <xacro:include filename="$(find sr_description)/hand/xacro/hand.urdf.xacro"/>
   <xacro:include filename="$(find sr_description)/other/xacro/gazebo.urdf.xacro"/>
-  <xacro:arg name="initial_hand_position" default="0.0 0.0 1.0"/>
+  <!-- <xacro:arg name="initial_hand_position"/> -->
+  <xacro:arg name="initial_hand_position" default="0.0 0.0 2.0"/>
   <xacro:arg name="initial_hand_orientation" default="1.57 -1.57 0.0"/>
   <xacro:arg name="hand_type" default="hand_e"/>
@@ -44,11 +45,14 @@
   <link name="world" />
   <xacro:if value="${'$(arg side)' == 'right'}">
-    <joint name="rh_world_joint" type="fixed">
-      <parent link="world" />
-      <child link="rh_forearm" />
-      <origin xyz="$(arg initial_hand_position)" rpy="$(arg initial_hand_orientation)" />
-      <!-- <origin xyz="0.0 0.0 1.0" rpy="0.0 0.0 0.0" /> -->
-    </joint>
-  </xacro:if>
+  <joint name="rh_world_joint" type="prismatic">
+    <parent link="world" />
+    <child link="rh_forearm" />
+    <origin xyz="$(arg initial_hand_position)" rpy="$(arg initial_hand_orientation)" />
+    <axis xyz="0 0 1"/> <!-- Assuming you want translation along the Z-axis -->
+    <limit lower="-3.14" upper="3.14" effort="1000" velocity="0.8"/> <!-- Adjust limits accordingly -->
+    <!-- <limit lower="-100" upper="100" velocity="0.8" effort="1000"/> -->
+    <!-- <joint name="rh_world_joint" type="fixed"> -->
+  </joint>
+</xacro:if>
   <xacro:if value="${'$(arg side)' == 'left'}">
     <joint name="lh_world_joint" type="fixed">
@@ -62,3 +66,7 @@
                  fingers="$(arg fingers)" tip_sensors="$(arg tip_sensors)" mid_sensors="$(arg mid_sensors)"
                  prox_sensors="$(arg prox_sensors)" palm_sensor="$(arg palm_sensor)" mounting_plate="$(arg mounting_plate)"/>
+<controller name="rh_world_joint_controller" type="position_controllers/JointPositionController">
+  <joint name="rh_world_joint"/>
+  <pid p="100.0" i="10.0" d="0.0"/>
+</controller>
 </robot>
